File: _autosave-FlowState.kicad_pcb (KiCad board)
At the start: 2 copper layers, 54.5 x 58.2 mm, 13 parts, among them J1 USB_C_Receptacle_USB2.0_16P, J2 Conn_01x04_Pin (CO2), J3 Conn_01x14_Pin(LCD), J4 Conn_01x03_Pin (SOIL), J5 Conn_01x04_Pin(SD), J6 Conn_01x02_Pin(Switch), U1 AMS1117-3.3, U2 ESP32-DEVKIT-V1

Commit message: heatsink
heatsink good now
Changed lines of the file:
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@@
 		(hatch edge 0.5)
 		(priority 1)
-		(connect_pads
-			(clearance 0.5)
+		(connect_pads yes
+			(clearance 0)
 		)
-		(min_thickness 0.25)
+		(min_thickness 0.025)
 		(filled_areas_thickness no)
-		(fill yes
+		(fill
 			(thermal_gap 0.5)
 			(thermal_bridge_width 0.5)
-			(smoothing fillet)
-			(radius 1)
 			(island_removal_mode 1)
 			(island_area_min 10)
@@
 		(polygon
 			(pts
-				(xy 30.2768 52.07) (xy 34.1376 52.07) (xy 34.1376 54.1528) (xy 30.2768 54.1528)
+				(xy 28.650538 51.3588) (xy 35.762538 51.3588) (xy 35.665013 58.2676) (xy 28.548938 58.2676)
 			)
 		)
