File: FlowState.kicad_pcb (KiCad board)
At the start: 2 copper layers, 54.5 x 58.2 mm, 13 parts, among them J1 USB_C_Receptacle_USB2.0_16P, J2 Conn_01x04_Pin (CO2), J3 Conn_01x14_Pin(LCD), J4 Conn_01x03_Pin (SOIL), J5 Conn_01x04_Pin(SD), J6 Conn_01x02_Pin(Switch), U1 AMS1117-3.3, U2 ESP32-DEVKIT-V1

Commit message: gerber, step, readme
did lots of stuff
Parts:
- added D1: 1N5819, Diode_THT:D_DO-41_SOD81_P10.16mm_Horizontal, F.Cu at (37.0, 63.9)
- moved J6 9.47 mm to (60.5, 57.9)
Routing:
- net GND: track 63.1 -> 73.4 mm
- net VCC_5V: track 103.5 -> 97.5 mm
- net USB_5V: track 50.1 -> 50.9 mm, vias 0 -> 1
Other:
- board size 54.5 x 58.2 mm -> 53 x 56.6 mm
